File: KiCAD/4_board/leverless_controller_4board.kicad_sch (KiCad schematic)
At the start: 41 parts

Commit message: 4 board DFM pass
Parts:
- added TP1, TP2: TestPoint, TestPoint:TestPoint_THTPad_1.0x1.0mm_Drill0.5mm, symbol Connector:TestPoint
Connections:
- new net +1V1: TP2.1
- new net +3.3V: TP1.1
