File: KiCAD/4_board/4board_a.kicad_pcb (KiCad board)
At the start: 2 copper layers, 95 x 99.5 mm, 68 parts, among them J1 USB_C_Receptacle_USB2.0_14P, J2 Conn_01x03_Socket, SW1 Memory Reset, SW17_W1 SW_Push, SW18_DOWN1 SW_Push, SW19_LEFT1 SW_Push, SW20_RIGHT1 SW_Push, SW8_DP1 SW_Push, U1 RP2040, U2 AMS1117-3.3_SOT223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

Commit message: 4 board DFM pass
Parts:
- added D1: LED, LED_SMD:LED_0603_1608Metric, F.Cu at (159.4, 33.4)
- added D2: LED, LED_SMD:LED_0603_1608Metric, F.Cu at (162.0, 33.4)
- added D3: LED, LED_SMD:LED_0603_1608Metric, F.Cu at (164.6, 33.4)
- added D4: LED, LED_SMD:LED_0603_1608Metric, F.Cu at (167.2, 33.4)
- added R9: 330, Resistor_SMD:R_0402_1005Metric, F.Cu at (159.5, 36.2)
- added TP1: TestPoint, TestPoint:TestPoint_THTPad_1.0x1.0mm_Drill0.5mm, F.Cu at (116.8, 35.6)
- added TP2: TestPoint, TestPoint:TestPoint_THTPad_1.0x1.0mm_Drill0.5mm, F.Cu at (130.9, 38.5)
- added TP3: TestPoint, TestPoint:TestPoint_Pad_D1.0mm, F.Cu at (143.4, 26.7)
- added TP4: TestPoint, TestPoint:TestPoint_Pad_D1.0mm, F.Cu at (141.1, 26.7)
- moved C16 1.68 mm to (138.7, 30.9)
- moved C15 1.64 mm to (144.0, 30.0), turned to 0 degrees
Connections:
- U1 pad 27: /Main/A2 -> /Main/P1
- U1 pad 28: /Main/A1 -> /Main/P2
- U1 pad 29: /Main/S1 -> /Main/P3
- U1 pad 30: /Main/S2 -> /Main/P4
- U1 pad 31: unconnected-(U1-GPIO20-Pad31) -> /Main/A2
- U1 pad 32: unconnected-(U1-GPIO21-Pad32) -> /Main/A1
- U1 pad 34: unconnected-(U1-GPIO22-Pad34) -> /Main/S1
- U1 pad 35: unconnected-(U1-GPIO23-Pad35) -> /Main/S2
- U1 pad 37: unconnected-(U1-GPIO25-Pad37) -> Net-(U1-GPIO25)
- U1 pad 39: unconnected-(U1-GPIO27_ADC1-Pad39) -> Net-(U1-GPIO27_ADC1)
Routing:
- net /Main/P4: track 0.00 -> 27.4 mm
- net /Main/P3: track 0.00 -> 23.8 mm
- net /Main/P2: track 0.00 -> 20.4 mm
- net /Main/P1: track 0.00 -> 17.6 mm
- net Net-(D1-K): track 0.00 -> 10.0 mm
- net Net-(U1-GPIO25): track 0.00 -> 7.94 mm
- net Net-(U1-GPIO27_ADC1): track 0.00 -> 7.08 mm
- net /Main/S1: track 53.9 -> 59.1 mm
- net +1V1: track 20.7 -> 25.8 mm
- net GND: track 208.8 -> 213.7 mm
- net /Main/S2: track 54.7 -> 58.9 mm
- net /Main/A1: track 54.0 -> 57.7 mm
- net /Main/A2: track 54.9 -> 58.0 mm
- net +3.3V: track 138.0 -> 141.1 mm
- net /Buttons/L3: track 0.00 -> 1.34 mm

Commit message: PCB Order Version
Parts:
- removed C16: 100n, Capacitor_SMD:C_0402_1005Metric
- removed C17, C18: 4.7u, Capacitor_SMD:C_0402_1005Metric
- removed SW17_W1, SW18_DOWN1, SW19_LEFT1, SW20_RIGHT1: SW_Push, PCM_Switch_Keyboard_Cherry_MX:SW_Cherry_MX_PCB_1.00u
- removed SW8_DP1: SW_Push, PCM_Switch_Keyboard_Cherry_MX:SW_Cherry_MX_PCB
- added SW17_W: SW_Push, PCM_Switch_Keyboard_Hotswap_Kailh:SW_Hotswap_Kailh_MX_1.00u, F.Cu at (174.1, 54.4)
- added SW18_DOWN: SW_Push, PCM_Switch_Keyboard_Hotswap_Kailh:SW_Hotswap_Kailh_MX_1.00u, F.Cu at (166.8, 72.0)
- added SW19_LEFT: SW_Push, PCM_Switch_Keyboard_Hotswap_Kailh:SW_Hotswap_Kailh_MX_1.00u, F.Cu at (149.2, 64.7)
- added SW20_RIGHT: SW_Push, PCM_Switch_Keyboard_Hotswap_Kailh:SW_Hotswap_Kailh_MX_1.00u, F.Cu at (182.9, 83.0)
- added SW8_DP: SW_Push, PCM_Switch_Keyboard_Hotswap_Kailh:SW_Hotswap_Kailh_MX, F.Cu at (117.0, 72.0)
- C1, C2: value 4.7u -> 10u
- D1, D2, D3, D4: footprint LED_SMD:LED_0603_1608Metric -> LED_SMD:LED_0805_2012Metric
- J1: footprint Fightstick_Library:USB_C_Receptacle_U262-161N-4BVC11 -> Fightstick_Library:USB_C_Receptacle_C6332272
- U2: footprint Package_TO_SOT_SMD:SOT-223-3_TabPin2 -> Fightstick_Library:LDO_AMS1117-3.3
- moved C11 10.8 mm to (138.7, 30.9)
- moved TP1 7.87 mm to (123.0, 30.8)
- moved C2 5.70 mm to (129.0, 35.5), turned to 90 degrees
- moved R9 1.87 mm to (159.0, 38.0)
- moved C1 1.11 mm to (126.0, 31.0)
- moved JP16 0.17 mm to (195.9, 115.0)
- moved JP14 0.14 mm to (195.9, 118.0)
- moved JP1 0.14 mm to (195.9, 47.2)
- moved JP10 0.14 mm to (195.9, 103.0)
- moved JP11 0.14 mm to (195.9, 106.0)
- moved JP12 0.14 mm to (195.9, 109.0)
- moved JP13 0.14 mm to (195.9, 112.0)
- moved JP2 0.14 mm to (195.9, 28.0)
- moved JP3 0.14 mm to (195.9, 30.8)
- moved JP4 0.14 mm to (195.9, 33.5)
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Connections:
- C2 pad 1: VBUS -> +3.3V
Routing:
- net +3.3V: track 141.1 -> 128.9 mm
- net L2: track 42.9 -> 48.2 mm, vias 0 -> 1
- net W: track 36.6 -> 33.1 mm, vias 0 -> 1
- net LEFT: track 23.1 -> 20.6 mm, vias 0 -> 1
- net DOWN: track 40.7 -> 38.2 mm, vias 0 -> 1
- net Net-(D1-K): track 10.0 -> 12.2 mm
- net GND: track 213.7 -> 212.0 mm, vias 15 -> 14
- net /Buttons/L3: track 1.34 -> 0.00 mm
- net RIGHT: track 61.7 -> 60.7 mm, vias 0 -> 1
