File: KiCAD/4_board/4board_b.kicad_pcb (KiCad board)
At the start: 2 copper layers, 92.5 x 99.5 mm, 29 parts, among them SW10_SHARE1 SW_Push, SW11_START1 SW_Push, SW14_PS1 SW_Push, SW15_TOUCHPAD1 SW_Push, SW2_LK1 SW_Push, SW3_MK1 SW_Push, SW4_LP1 SW_Push, SW5_MP1 SW_Push, SW6_DI1 SW_Push, SW7_HP1 SW_Push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

Commit message: 4 board DFM pass
Parts:
- SW10_SHARE1, SW11_START1, SW14_PS1, SW15_TOUCHPAD1: footprint Button_Switch_THT:SW_SPST_Omron_B3F-40xx -> Fightstick_Library:SW_SPST_6x12
Changed lines of the file:
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@@
 		)
 	)
-	(footprint "Button_Switch_THT:SW_SPST_Omron_B3F-40xx"
+	(footprint "Fightstick_Library:SW_SPST_6x12"
 		(layer "F.Cu")
 		(at 184.765 35.25 90)
@@
 		(tags "tactile switch THT button push B3F-4000 B3F-4050 B3F-4005 B3F-4055  ")
 		(property "Reference" "SW15_TOUCHPAD1"
-			(at 6.25 -4.5 90)
-			(unlocked yes)
+			(at 6.25 -4.5 -90)
 			(layer "F.SilkS")
 			(effects
@@
 		(property "Value" "SW_Push"
 			(at 6.25 10.8 90)
-			(unlocked yes)
-			(layer "F.Fab")
-			(effects
-				(font
-					(size 1 1)
-					(thickness 0.15)
-				)
-			)
-		)
-		(property "Footprint" "Button_Switch_THT:SW_SPST_Omron_B3F-40xx"
+			(layer "F.Fab")
+			(effects
+				(font
+					(size 1 1)
+					(thickness 0.15)
+				)
+			)
+		)
+		(property "Footprint" "Fightstick_Library:SW_SPST_6x12"
 			(at 0 0 90)
 			(unlocked yes)
@@
 				)
 			)
-		)
-		(pad "" np_thru_hole circle
-			(at 6.25 -2 90)
-			(size 1.8 1.8)
-			(drill 1.8)
-			(layers "F&B.Cu" "*.Mask")
-		)
-		(pad "" np_thru_hole circle
-			(at 6.25 7 90)
-			(size 1.8 1.8)
-			(drill 1.8)
-			(layers "F&B.Cu" "*.Mask")
 		)
 		(pad "1" thru_hole oval
@@
 		)
 	)
-	(footprint "Button_Switch_THT:SW_SPST_Omron_B3F-40xx"
+	(footprint "Fightstick_Library:SW_SPST_6x12"
 		(layer "F.Cu")
 		(at 139.765 35.25 90)
@@
 		(tags "tactile switch THT button push B3F-4000 B3F-4050 B3F-4005 B3F-4055  ")
 		(property "Reference" "SW11_START1"
-			(at 6.25 -4.5 90)
-			(unlocked yes)
+			(at 6.25 -4.5 -90)
 			(layer "F.SilkS")
 			(effects
@@
 		(property "Value" "SW_Push"
 			(at 6.25 10.8 90)
-			(unlocked yes)
-			(layer "F.Fab")
-			(effects
-				(font
-					(size 1 1)
-					(thickness 0.15)
-				)
-			)
-		)
-		(property "Footprint" "Button_Switch_THT:SW_SPST_Omron_B3F-40xx"
+			(layer "F.Fab")
+			(effects
+				(font
+					(size 1 1)
+					(thickness 0.15)
+				)
+			)
+		)
+		(property "Footprint" "Fightstick_Library:SW_SPST_6x12"
 			(at 0 0 90)
 			(unlocked yes)
@@
 				)
 			)
-		)
-		(pad "" np_thru_hole circle
-			(at 6.25 -2 90)
-			(size 1.8 1.8)
-			(drill 1.8)
-			(layers "F&B.Cu" "*.Mask")
-		)
-		(pad "" np_thru_hole circle
-			(at 6.25 7 90)
-			(size 1.8 1.8)
-			(drill 1.8)
-			(layers "F&B.Cu" "*.Mask")
 		)
 		(pad "1" thru_hole oval
@@
 		)
 	)
-	(footprint "Button_Switch_THT:SW_SPST_Omron_B3F-40xx"
+	(footprint "Fightstick_Library:SW_SPST_6x12"
 		(layer "F.Cu")
 		(at 154.765 35.25 90)
@@
 		(tags "tactile switch THT button push B3F-4000 B3F-4050 B3F-4005 B3F-4055  ")
 		(property "Reference" "SW10_SHARE1"
-			(at 6.25 -4.5 90)
-			(unlocked yes)
+			(at 6.25 -4.5 -90)
 			(layer "F.SilkS")
 			(effects
@@
 		(property "Value" "SW_Push"
 			(at 6.25 10.8 90)
-			(unlocked yes)
-			(layer "F.Fab")
-			(effects
-				(font
-					(size 1 1)
-					(thickness 0.15)
-				)
-			)
-		)
-		(property "Footprint" "Button_Switch_THT:SW_SPST_Omron_B3F-40xx"
+			(layer "F.Fab")
+			(effects
+				(font
+					(size 1 1)
+					(thickness 0.15)
+				)
+			)
+		)
+		(property "Footprint" "Fightstick_Library:SW_SPST_6x12"
 			(at 0 0 90)
 			(unlocked yes)
@@
 				)
 			)
-		)
-		(pad "" np_thru_hole circle
-			(at 6.25 -2 90)
-			(size 1.8 1.8)
-			(drill 1.8)
-			(layers "F&B.Cu" "*.Mask")
-		)
-		(pad "" np_thru_hole circle
-			(at 6.25 7 90)
-			(size 1.8 1.8)
-			(drill 1.8)
-			(layers "F&B.Cu" "*.Mask")
 		)
 		(pad "1" thru_hole oval
@@
 		)
 	)
-	(footprint "Button_Switch_THT:SW_SPST_Omron_B3F-40xx"
+	(footprint "Fightstick_Library:SW_SPST_6x12"
 		(layer "F.Cu")
 		(at 169.765 35.25 90)
@@
 		(tags "tactile switch THT button push B3F-4000 B3F-4050 B3F-4005 B3F-4055  ")
 		(property "Reference" "SW14_PS1"
-			(at 6.25 -4.5 90)
-			(unlocked yes)
+			(at 6.25 -4.5 -90)
 			(layer "F.SilkS")
 			(effects
@@
 		(property "Value" "SW_Push"
 			(at 6.25 10.8 90)
-			(unlocked yes)
-			(layer "F.Fab")
-			(effects
-				(font
-					(size 1 1)
-					(thickness 0.15)
-				)
-			)
-		)
-		(property "Footprint" "Button_Switch_THT:SW_SPST_Omron_B3F-40xx"
+			(layer "F.Fab")
+			(effects
+				(font
+					(size 1 1)
+					(thickness 0.15)
+				)
+			)
+		)
+		(property "Footprint" "Fightstick_Library:SW_SPST_6x12"
 			(at 0 0 90)
 			(unlocked yes)
@@
 			)
 		)
-		(pad "" np_thru_hole circle
-			(at 6.25 -2 90)
-			(size 1.8 1.8)
-			(drill 1.8)
-			(layers "F&B.Cu" "*.Mask")
-		)
-		(pad "" np_thru_hole circle
-			(at 6.25 7 90)
-			(size 1.8 1.8)
-			(drill 1.8)
-			(layers "F&B.Cu" "*.Mask")
-		)
 		(pad "1" thru_hole oval

Commit message: PCB Order Version
Parts:
- removed SW10_SHARE1, SW11_START1, SW14_PS1, SW15_TOUCHPAD1: SW_Push, Fightstick_Library:SW_SPST_6x12
- removed SW2_LK1, SW3_MK1, SW4_LP1, SW5_MP1, SW6_DI1, SW7_HP1, SW9_HK1: SW_Push, PCM_Switch_Keyboard_Cherry_MX:SW_Cherry_MX_PCB
- added SW10_SHARE: SW_Push, PCM_Switch_Keyboard_Cherry_MX:SW_Cherry_MX_PCB, F.Cu at (154.7, 29.1)
- added SW11_START: SW_Push, PCM_Switch_Keyboard_Cherry_MX:SW_Cherry_MX_PCB, F.Cu at (139.2, 29.1)
- added SW14_PS: SW_Push, PCM_Switch_Keyboard_Cherry_MX:SW_Cherry_MX_PCB, F.Cu at (170.2, 29.1)
- added SW15_TOUCHPAD: SW_Push, PCM_Switch_Keyboard_Cherry_MX:SW_Cherry_MX_PCB, F.Cu at (185.7, 29.1)
- added SW2_LK: SW_Push, PCM_Switch_Keyboard_Hotswap_Kailh:SW_Hotswap_Kailh_MX, F.Cu at (117.2, 98.0)
- added SW3_MK: SW_Push, PCM_Switch_Keyboard_Hotswap_Kailh:SW_Hotswap_Kailh_MX, F.Cu at (142.2, 84.0)
- added SW4_LP: SW_Push, PCM_Switch_Keyboard_Hotswap_Kailh:SW_Hotswap_Kailh_MX, F.Cu at (117.2, 69.0)
- added SW5_MP: SW_Push, PCM_Switch_Keyboard_Hotswap_Kailh:SW_Hotswap_Kailh_MX, F.Cu at (142.2, 55.0)
- added SW6_DI: SW_Push, PCM_Switch_Keyboard_Hotswap_Kailh:SW_Hotswap_Kailh_MX, F.Cu at (117.3, 40.0)
- added SW7_HP: SW_Push, PCM_Switch_Keyboard_Hotswap_Kailh:SW_Hotswap_Kailh_MX, F.Cu at (171.2, 55.0)
- added SW9_HK: SW_Push, PCM_Switch_Keyboard_Hotswap_Kailh:SW_Hotswap_Kailh_MX, F.Cu at (171.2, 84.0)
- moved JP15 0.11 mm to (102.3, 41.2)
- moved JP17 0.11 mm to (102.3, 97.0)
- moved JP18 0.11 mm to (102.3, 100.0)
- moved JP19 0.11 mm to (102.3, 103.0)
- moved JP20 0.11 mm to (102.3, 106.0)
- moved JP21 0.11 mm to (102.3, 22.0)
- moved JP22 0.11 mm to (102.3, 24.8)
- moved JP23 0.11 mm to (102.3, 27.5)
- moved JP24 0.11 mm to (102.3, 30.2)
- moved JP25 0.11 mm to (102.3, 33.0)
- moved JP26 0.11 mm to (102.3, 35.8)
- moved JP27 0.11 mm to (102.3, 38.5)
Routing:
- net GND: track 382.5 -> 307.0 mm
- net /Buttons/A1: track 84.5 -> 68.5 mm
- net /Buttons/A2: track 98.8 -> 83.3 mm
- net /Buttons/S2: track 49.7 -> 34.5 mm
- net /Buttons/S1: track 65.5 -> 54.1 mm
- net /Buttons/L1: track 13.0 -> 9.28 mm, vias 0 -> 1
- net /Buttons/B2: track 44.8 -> 41.5 mm, vias 0 -> 1
- net /Buttons/B4: track 41.3 -> 38.1 mm, vias 0 -> 1
- net /Buttons/R1: track 71.4 -> 68.5 mm, vias 0 -> 1
- net /Buttons/R2: track 76.3 -> 73.7 mm, vias 0 -> 1
- net /Buttons/B3: track 36.1 -> 33.5 mm, vias 0 -> 1
- net /Buttons/B1: track 15.8 -> 13.5 mm, vias 0 -> 1
Other:
- board text removed: "TODO Move these buttons further away from the rest"
