File: KiCAD/4_board/4board_c.kicad_pcb (KiCad board)
At the start: 2 copper layers, 20.7 x 50.5 mm, 21 parts, among them SW12_THROW1 SW_Push

Commit message: PCB Order Version
Parts:
- removed SW12_THROW1: SW_Push, PCM_Switch_Keyboard_Cherry_MX:SW_Cherry_MX_PCB
- added SW12_THROW: SW_Push, PCM_Switch_Keyboard_Hotswap_Kailh:SW_Hotswap_Kailh_MX, F.Cu at (148.9, 54.4)
- moved JP15 0.13 mm to (158.8, 41.2)
- moved JP21 0.13 mm to (158.8, 22.0)
- moved JP22 0.13 mm to (158.8, 24.8)
- moved JP23 0.13 mm to (158.8, 27.5)
- moved JP24 0.13 mm to (158.8, 30.2)
- moved JP25 0.13 mm to (158.8, 33.0)
- moved JP26 0.13 mm to (158.8, 35.8)
- moved JP27 0.13 mm to (158.8, 38.5)
- moved JP1 0.11 mm to (138.2, 41.2)
- moved JP2 0.11 mm to (138.2, 22.0)
- moved JP3 0.11 mm to (138.2, 24.8)
- moved JP4 0.11 mm to (138.2, 27.5)
- moved JP5 0.11 mm to (138.2, 30.2)
- moved JP6 0.11 mm to (138.2, 33.0)
- moved JP7 0.11 mm to (138.2, 35.8)
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Routing:
- net /Buttons/L3: track 10.4 -> 9.05 mm, vias 0 -> 1
- net GND: track 28.0 -> 26.9 mm, vias 0 -> 1
