File: KiCAD/4_board/4board_d.kicad_pcb (KiCad board)
At the start: 2 copper layers, 41 x 46 mm, 14 parts, among them SW16_SPACE1 SW_Push

Commit message: PCB Order Version
Parts:
- removed SW16_SPACE1: SW_Push, PCM_Switch_Keyboard_Cherry_MX:SW_Cherry_MX_PCB
- added SW16_SPACE: SW_Push, PCM_Switch_Keyboard_Hotswap_Kailh:SW_Hotswap_Kailh_MX, F.Cu at (148.4, 54.8)
- moved JP17 0.15 mm to (157.8, 21.8)
- moved JP18 0.15 mm to (157.8, 24.8)
- moved JP19 0.15 mm to (157.8, 27.8)
- moved JP20 0.15 mm to (157.8, 30.8)
- moved JP10 0.11 mm to (137.2, 21.8)
- moved JP11 0.11 mm to (137.2, 24.8)
- moved JP12 0.11 mm to (137.2, 27.8)
- moved JP13 0.11 mm to (137.2, 30.8)
- moved JP14 0.11 mm to (137.2, 36.8)
- moved JP16 0.11 mm to (137.2, 33.8)
Routing:
- net GND: track 21.7 -> 24.0 mm, vias 0 -> 1
- net /Buttons/SPACE: track 18.4 -> 17.0 mm, vias 0 -> 1
Other:
- board text removed: "JP17"
- board text removed: "JP18"
- board text removed: "JP19"
- board text removed: "JP20"
