File: KiCAD/4_board/Buttons.kicad_sch (KiCad schematic)
At the start: 18 parts, among them SW10_SHARE1 SW_Push, SW11_START1 SW_Push, SW12_THROW1 SW_Push, SW14_PS1 SW_Push, SW15_TOUCHPAD1 SW_Push, SW16_SPACE1 SW_Push, SW17_W1 SW_Push, SW18_DOWN1 SW_Push, SW19_LEFT1 SW_Push, SW20_RIGHT1 SW_Push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

Commit message: 4 board DFM pass
Parts:
- SW10_SHARE1, SW11_START1, SW14_PS1, SW15_TOUCHPAD1: footprint Button_Switch_THT:SW_SPST_Omron_B3F-40xx -> Fightstick_Library:SW_SPST_6x12
Changed lines of the file:
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@@
 			)
 		)
-		(property "Footprint" "Button_Switch_THT:SW_SPST_Omron_B3F-40xx"
+		(property "Footprint" "Fightstick_Library:SW_SPST_6x12"
 			(at 34.29 173.99 0)
 			(effects
@@
 			)
 		)
-		(property "Footprint" "Button_Switch_THT:SW_SPST_Omron_B3F-40xx"
+		(property "Footprint" "Fightstick_Library:SW_SPST_6x12"
 			(at 34.29 156.21 0)
 			(effects
@@
 			)
 		)
-		(property "Footprint" "Button_Switch_THT:SW_SPST_Omron_B3F-40xx"
+		(property "Footprint" "Fightstick_Library:SW_SPST_6x12"
 			(at 71.12 69.85 0)
 			(effects
@@
 			)
 		)
-		(property "Footprint" "Button_Switch_THT:SW_SPST_Omron_B3F-40xx"
+		(property "Footprint" "Fightstick_Library:SW_SPST_6x12"
 			(at 69.85 53.34 0)
 			(effects

Commit message: PCB Order Version
Parts:
- SW10_SHARE1, SW11_START1, SW14_PS1, SW15_TOUCHPAD1: footprint Fightstick_Library:SW_SPST_6x12 -> PCM_Switch_Keyboard_Cherry_MX:SW_Cherry_MX_PCB
- SW12_THROW1, SW16_SPACE1, SW2_LK1, SW3_MK1, SW4_LP1, SW5_MP1, SW6_DI1, SW7_HP1, SW8_DP1, SW9_HK1: footprint PCM_Switch_Keyboard_Cherry_MX:SW_Cherry_MX_PCB -> PCM_Switch_Keyboard_Hotswap_Kailh:SW_Hotswap_Kailh_MX
- SW17_W1, SW18_DOWN1, SW19_LEFT1, SW20_RIGHT1: footprint PCM_Switch_Keyboard_Cherry_MX:SW_Cherry_MX_PCB_1.00u -> PCM_Switch_Keyboard_Hotswap_Kailh:SW_Hotswap_Kailh_MX_1.00u
Changed lines of the file:
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@@
 			)
 		)
-		(property "Footprint" "PCM_Switch_Keyboard_Cherry_MX:SW_Cherry_MX_PCB_1.00u"
+		(property "Footprint" "PCM_Switch_Keyboard_Hotswap_Kailh:SW_Hotswap_Kailh_MX_1.00u"
 			(at 71.12 120.65 0)
 			(effects
@@
 			)
 		)
-		(property "Footprint" "PCM_Switch_Keyboard_Cherry_MX:SW_Cherry_MX_PCB"
+		(property "Footprint" "PCM_Switch_Keyboard_Hotswap_Kailh:SW_Hotswap_Kailh_MX"
 			(at 34.29 69.85 0)
 			(effects
@@
 			)
 		)
-		(property "Footprint" "PCM_Switch_Keyboard_Cherry_MX:SW_Cherry_MX_PCB_1.00u"
+		(property "Footprint" "PCM_Switch_Keyboard_Hotswap_Kailh:SW_Hotswap_Kailh_MX_1.00u"
 			(at 71.12 156.21 0)
 			(effects
@@
 			)
 		)
-		(property "Footprint" "PCM_Switch_Keyboard_Cherry_MX:SW_Cherry_MX_PCB_1.00u"
+		(property "Footprint" "PCM_Switch_Keyboard_Hotswap_Kailh:SW_Hotswap_Kailh_MX_1.00u"
 			(at 71.12 102.87 0)
 			(effects
@@
 			)
 		)
-		(property "Footprint" "Fightstick_Library:SW_SPST_6x12"
+		(property "Footprint" "PCM_Switch_Keyboard_Cherry_MX:SW_Cherry_MX_PCB"
 			(at 34.29 173.99 0)
 			(effects
@@
 			)
 		)
-		(property "Footprint" "PCM_Switch_Keyboard_Cherry_MX:SW_Cherry_MX_PCB"
+		(property "Footprint" "PCM_Switch_Keyboard_Hotswap_Kailh:SW_Hotswap_Kailh_MX"
 			(at 71.12 85.09 0)
 			(effects
@@
 			)
 		)
-		(property "Footprint" "PCM_Switch_Keyboard_Cherry_MX:SW_Cherry_MX_PCB"
+		(property "Footprint" "PCM_Switch_Keyboard_Hotswap_Kailh:SW_Hotswap_Kailh_MX"
 			(at 69.85 20.32 0)
 			(effects
@@
 			)
 		)
-		(property "Footprint" "PCM_Switch_Keyboard_Cherry_MX:SW_Cherry_MX_PCB"
+		(property "Footprint" "PCM_Switch_Keyboard_Hotswap_Kailh:SW_Hotswap_Kailh_MX"
 			(at 34.29 36.83 0)
 			(effects
@@
 			)
 		)
-		(property "Footprint" "Fightstick_Library:SW_SPST_6x12"
+		(property "Footprint" "PCM_Switch_Keyboard_Cherry_MX:SW_Cherry_MX_PCB"
 			(at 34.29 156.21 0)
 			(effects
@@
 			)
 		)
-		(property "Footprint" "PCM_Switch_Keyboard_Cherry_MX:SW_Cherry_MX_PCB"
+		(property "Footprint" "PCM_Switch_Keyboard_Hotswap_Kailh:SW_Hotswap_Kailh_MX"
 			(at 34.29 53.34 0)
 			(effects
@@
 			)
 		)
-		(property "Footprint" "PCM_Switch_Keyboard_Cherry_MX:SW_Cherry_MX_PCB"
+		(property "Footprint" "PCM_Switch_Keyboard_Hotswap_Kailh:SW_Hotswap_Kailh_MX"
 			(at 34.29 138.43 0)
 			(effects
@@
 			)
 		)
-		(property "Footprint" "Fightstick_Library:SW_SPST_6x12"
+		(property "Footprint" "PCM_Switch_Keyboard_Cherry_MX:SW_Cherry_MX_PCB"
 			(at 71.12 69.85 0)
 			(effects
@@
 			)
 		)
-		(property "Footprint" "Fightstick_Library:SW_SPST_6x12"
+		(property "Footprint" "PCM_Switch_Keyboard_Cherry_MX:SW_Cherry_MX_PCB"
 			(at 69.85 53.34 0)
 			(effects
@@
 			)
 		)
-		(property "Footprint" "PCM_Switch_Keyboard_Cherry_MX:SW_Cherry_MX_PCB"
+		(property "Footprint" "PCM_Switch_Keyboard_Hotswap_Kailh:SW_Hotswap_Kailh_MX"
 			(at 34.29 120.65 0)
 			(effects
@@
 			)
 		)
-		(property "Footprint" "PCM_Switch_Keyboard_Cherry_MX:SW_Cherry_MX_PCB"
+		(property "Footprint" "PCM_Switch_Keyboard_Hotswap_Kailh:SW_Hotswap_Kailh_MX"
 			(at 34.29 20.32 0)
 			(effects
@@
 			)
 		)
-		(property "Footprint" "PCM_Switch_Keyboard_Cherry_MX:SW_Cherry_MX_PCB"
+		(property "Footprint" "PCM_Switch_Keyboard_Hotswap_Kailh:SW_Hotswap_Kailh_MX"
 			(at 34.29 102.87 0)
 			(effects
@@
 			)
 		)
-		(property "Footprint" "PCM_Switch_Keyboard_Cherry_MX:SW_Cherry_MX_PCB_1.00u"
+		(property "Footprint" "PCM_Switch_Keyboard_Hotswap_Kailh:SW_Hotswap_Kailh_MX_1.00u"
 			(at 71.12 138.43 0)
 			(effects
@@
 			)
 		)
-		(property "Footprint" "PCM_Switch_Keyboard_Cherry_MX:SW_Cherry_MX_PCB"
+		(property "Footprint" "PCM_Switch_Keyboard_Hotswap_Kailh:SW_Hotswap_Kailh_MX"
 			(at 34.29 85.09 0)
 			(effects
