File: KiCAD/4_board/Main.kicad_sch (KiCad schematic)
At the start: 33 parts, among them J1 USB_C_Receptacle_USB2.0_14P, J2 Conn_01x03_Socket, SW1 Memory Reset, U1 RP2040, U2 AMS1117-3.3_SOT223, U3 W25Q128JVSIQ, Y1 12 mhz crystal

Commit message: 4 board DFM pass
Parts:
- added D1, D2, D3, D4: LED, LED_SMD:LED_0603_1608Metric, symbol Device:LED
- added R9: 330, Resistor_SMD:R_0402_1005Metric, symbol Device:R
- added TP3, TP4: TestPoint, TestPoint:TestPoint_Pad_D1.0mm, symbol Connector:TestPoint
- C1, C17, C18, C2: LCSC C15525 -> C23733
Connections:
- net A1: now also U1.32 (GPIO21); no longer U1.28 (GPIO17)
- net A2: now also U1.31 (GPIO20); no longer U1.27 (GPIO16)
- net GND: now also R9.2
- net S1: now also U1.34 (GPIO22); no longer U1.29 (GPIO18)
- net S2: now also U1.35 (GPIO23); no longer U1.30 (GPIO19)
- net at U1.37 (GPIO25): now also TP3.1
- net at U1.39 (GPIO27_ADC1): now also TP4.1
- new net: D1.1 (K), D2.1 (K), D3.1 (K), D4.1 (K), R9.1
- new net P1: D1.2 (A), U1.27 (GPIO16)
- new net P2: D2.2 (A), U1.28 (GPIO17)
- new net P3: D3.2 (A), U1.29 (GPIO18)
- new net P4: D4.2 (A), U1.30 (GPIO19)
- no-connect marks 14 -> 8
Other:
- note added: "LEDs"

Commit message: PCB Order Version
Parts:
- removed C11: 100n, Capacitor_SMD:C_0402_1005Metric, symbol Device:C
- removed C17, C18: 4.7u, Capacitor_SMD:C_0402_1005Metric, symbol Device:C
- C1, C2: value 4.7u -> 10u; LCSC C23733 -> C15525
- D1, D2, D3, D4: footprint LED_SMD:LED_0603_1608Metric -> LED_SMD:LED_0805_2012Metric
- J1: footprint Fightstick_Library:USB_C_Receptacle_U262-161N-4BVC11 -> Fightstick_Library:USB_C_Receptacle_C6332272
- R6: now not fitted
- U2: footprint Package_TO_SOT_SMD:SOT-223-3_TabPin2 -> Fightstick_Library:LDO_AMS1117-3.3
- renumbered C16 to C11
Connections:
- net +3.3V: now also C2.1
- net VBUS: no longer C2.1
Other:
- note added: "Tie RUN pin to IOVDD for no external resets"
- note removed: "Tie RUN pin to IOVDD for now external resets"
- moved on the sheet: C1, C11, C2
