File: KiCAD/4_board/leverless_controller_4board.kicad_pcb (KiCad board)
At the start: 2 copper layers, 208.5 x 127.2 mm, 105 parts, among them J1 USB_C_Receptacle_USB2.0_14P, J2 Conn_01x03_Socket, SW1 Memory Reset, SW10_SHARE1 SW_Push, SW11_START1 SW_Push, SW12_THROW1 SW_Push, SW14_PS1 SW_Push, SW15_TOUCHPAD1 SW_Push, SW16_SPACE1 SW_Push, SW17_W1 SW_Push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

Commit message: 4 board DFM pass
Parts:
- added D1: LED, LED_SMD:LED_0603_1608Metric, F.Cu at (102.4, 33.4)
- added D2: LED, LED_SMD:LED_0603_1608Metric, F.Cu at (105.0, 33.4)
- added D3: LED, LED_SMD:LED_0603_1608Metric, F.Cu at (107.6, 33.4)
- added D4: LED, LED_SMD:LED_0603_1608Metric, F.Cu at (110.2, 33.4)
- added R9: 330, Resistor_SMD:R_0402_1005Metric, F.Cu at (102.5, 36.2)
- added TP1: TestPoint, TestPoint:TestPoint_THTPad_1.0x1.0mm_Drill0.5mm, F.Cu at (59.8, 35.6)
- added TP2: TestPoint, TestPoint:TestPoint_THTPad_1.0x1.0mm_Drill0.5mm, F.Cu at (73.9, 38.5)
- added TP3: TestPoint, TestPoint:TestPoint_Pad_D1.0mm, F.Cu at (86.4, 26.7)
- added TP4: TestPoint, TestPoint:TestPoint_Pad_D1.0mm, F.Cu at (84.1, 26.7)
- SW10_SHARE1, SW11_START1, SW14_PS1, SW15_TOUCHPAD1: footprint Button_Switch_THT:SW_SPST_Omron_B3F-40xx -> Fightstick_Library:SW_SPST_6x12
- moved C16 1.68 mm to (81.7, 30.9)
- moved C15 1.64 mm to (87.0, 30.0), turned to 0 degrees
Connections:
- U1 pad 27: /Main/A2 -> /Main/P1
- U1 pad 28: /Main/A1 -> /Main/P2
- U1 pad 29: /Main/S1 -> /Main/P3
- U1 pad 30: /Main/S2 -> /Main/P4
- U1 pad 31: unconnected-(U1-GPIO20-Pad31) -> /Main/A2
- U1 pad 32: unconnected-(U1-GPIO21-Pad32) -> /Main/A1
- U1 pad 34: unconnected-(U1-GPIO22-Pad34) -> /Main/S1
- U1 pad 35: unconnected-(U1-GPIO23-Pad35) -> /Main/S2
- U1 pad 37: unconnected-(U1-GPIO25-Pad37) -> Net-(U1-GPIO25)
- U1 pad 39: unconnected-(U1-GPIO27_ADC1-Pad39) -> Net-(U1-GPIO27_ADC1)
Routing:
- net /Main/P4: track 0.00 -> 27.4 mm
- net /Main/P3: track 0.00 -> 23.8 mm
- net /Main/P2: track 0.00 -> 20.4 mm
- net /Main/P1: track 0.00 -> 17.6 mm
- net Net-(D1-K): track 0.00 -> 10.0 mm
- net Net-(U1-GPIO25): track 0.00 -> 7.94 mm
- net Net-(U1-GPIO27_ADC1): track 0.00 -> 7.08 mm
- net /Main/S1: track 53.9 -> 59.1 mm
- net +1V1: track 20.7 -> 25.8 mm
- net GND: track 641.0 -> 645.9 mm
- net /Main/S2: track 54.7 -> 58.9 mm
- net /Main/A1: track 54.0 -> 57.7 mm
- net /Main/A2: track 54.9 -> 58.0 mm
- net +3.3V: track 138.0 -> 141.1 mm

Commit message: PCB Order Version
Parts:
- removed the C11 at (71.9, 35.4)
- removed C17, C18: 4.7u, Capacitor_SMD:C_0402_1005Metric
- C1, C2: value 4.7u -> 10u
- D1, D2, D3, D4: footprint LED_SMD:LED_0603_1608Metric -> LED_SMD:LED_0805_2012Metric
- J1: footprint Fightstick_Library:USB_C_Receptacle_U262-161N-4BVC11 -> Fightstick_Library:USB_C_Receptacle_C6332272
- SW10_SHARE1, SW11_START1, SW14_PS1, SW15_TOUCHPAD1: footprint Fightstick_Library:SW_SPST_6x12 -> PCM_Switch_Keyboard_Cherry_MX:SW_Cherry_MX_PCB
- SW12_THROW1, SW16_SPACE1, SW2_LK1, SW3_MK1, SW4_LP1, SW5_MP1, SW6_DI1, SW7_HP1, SW8_DP1, SW9_HK1: footprint PCM_Switch_Keyboard_Cherry_MX:SW_Cherry_MX_PCB -> PCM_Switch_Keyboard_Hotswap_Kailh:SW_Hotswap_Kailh_MX
- SW17_W1, SW18_DOWN1, SW19_LEFT1, SW20_RIGHT1: footprint PCM_Switch_Keyboard_Cherry_MX:SW_Cherry_MX_PCB_1.00u -> PCM_Switch_Keyboard_Hotswap_Kailh:SW_Hotswap_Kailh_MX_1.00u
- U2: footprint Package_TO_SOT_SMD:SOT-223-3_TabPin2 -> Fightstick_Library:LDO_AMS1117-3.3
- moved TP1 7.87 mm to (66.0, 30.8)
- moved SW15_TOUCHPAD1 6.25 mm to (243.5, 35.1), turned to 0 degrees
- moved SW11_START1 6.19 mm to (197.0, 35.1), turned to 0 degrees
- moved SW14_PS1 6.19 mm to (228.0, 35.1), turned to 0 degrees
- moved SW10_SHARE1 6.17 mm to (212.5, 35.1), turned to 0 degrees
- moved C2 5.70 mm to (72.0, 35.5), turned to 90 degrees
- moved R9 1.87 mm to (102.0, 38.0)
- moved C1 1.11 mm to (69.0, 31.0)
- turned H3 to 180 degrees
- renumbered C16 to C11
Connections:
- C2 pad 1: VBUS -> +3.3V
Routing:
- net GND: track 645.9 -> 570.3 mm, vias 16 -> 17
- net /Buttons/A1: track 84.5 -> 68.5 mm
- net /Buttons/A2: track 98.8 -> 83.3 mm
- net /Buttons/S2: track 49.7 -> 34.5 mm
- net +3.3V: track 141.1 -> 128.9 mm
- net /Buttons/S1: track 65.5 -> 54.1 mm
- net L2: track 42.9 -> 48.2 mm, vias 0 -> 1
- net /Buttons/L1: track 13.0 -> 9.28 mm, vias 0 -> 1
- net W: track 36.6 -> 33.1 mm, vias 0 -> 1
- net /Buttons/B2: track 44.8 -> 41.5 mm, vias 0 -> 1
- net /Buttons/B4: track 41.3 -> 38.1 mm, vias 0 -> 1
- net /Buttons/R1: track 71.4 -> 68.5 mm, vias 0 -> 1
- net /Buttons/R2: track 76.3 -> 73.7 mm, vias 0 -> 1
- net /Buttons/B3: track 36.1 -> 33.5 mm, vias 0 -> 1
- net LEFT: track 23.1 -> 20.6 mm, vias 0 -> 1
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Other:
- board text removed: "TODO Move these buttons further away from the rest"
