File: KiCAD/4_board/panel_1.kicad_pcb (KiCad board)
At the start: 2 copper layers, 95 x 99.5 mm, 93 parts, among them J1 USB_C_Receptacle_USB2.0_14P, J2 Conn_01x03_Socket, SW1 Memory Reset, SW16_SPACE1 SW_Push, SW17_W1 SW_Push, SW18_DOWN1 SW_Push, SW19_LEFT1 SW_Push, SW20_RIGHT1 SW_Push, SW8_DP1 SW_Push, U1 RP2040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

Commit message: 4 board DFM pass
Parts:
- removed the ? at (161.9, 40.7)
- removed the ? at (162.9, 41.7)
- removed the ? at (161.9, 42.8)
- removed the ? at (162.9, 40.7)
- removed the ? at (162.9, 42.8)
- removed the ? at (160.9, 42.8)
- removed the ? at (160.9, 41.7)
- removed the ? at (160.9, 40.7)
- removed the ? at (161.9, 41.7)
- removed SW17_W1, SW18_DOWN1, SW19_LEFT1, SW20_RIGHT1: SW_Push, PCM_Switch_Keyboard_Cherry_MX:SW_Cherry_MX_PCB_1.00u
- removed SW8_DP1: SW_Push, PCM_Switch_Keyboard_Cherry_MX:SW_Cherry_MX_PCB
- added ?: , , F.Cu at (83.7, 36.8)
- added ?: , , F.Cu at (84.7, 36.8)
- added ?: , , F.Cu at (85.7, 35.8)
- added ?: , , F.Cu at (85.7, 37.9)
- added ?: , , F.Cu at (85.7, 36.8)
- added ?: , , F.Cu at (83.7, 37.9)
- added ?: , , F.Cu at (83.7, 35.8)
- added ?: , , F.Cu at (84.7, 35.8)
- added ?: , , F.Cu at (84.7, 37.9)
- added D1: LED, LED_SMD:LED_0603_1608Metric, F.Cu at (102.4, 33.4)
- added D2: LED, LED_SMD:LED_0603_1608Metric, F.Cu at (105.0, 33.4)
- added D3: LED, LED_SMD:LED_0603_1608Metric, F.Cu at (107.6, 33.4)
- added D4: LED, LED_SMD:LED_0603_1608Metric, F.Cu at (110.2, 33.4)
- added R9: 330, Resistor_SMD:R_0402_1005Metric, F.Cu at (102.5, 36.2)
- added SW17_W: SW_Push, PCM_Switch_Keyboard_Cherry_MX:SW_Cherry_MX_PCB_1.00u, F.Cu at (117.1, 54.4)
- added SW18_DOWN: SW_Push, PCM_Switch_Keyboard_Cherry_MX:SW_Cherry_MX_PCB_1.00u, F.Cu at (109.8, 72.0)
- added SW19_LEFT: SW_Push, PCM_Switch_Keyboard_Cherry_MX:SW_Cherry_MX_PCB_1.00u, F.Cu at (92.2, 64.7)
- added SW20_RIGHT: SW_Push, PCM_Switch_Keyboard_Cherry_MX:SW_Cherry_MX_PCB_1.00u, F.Cu at (125.9, 83.0)
- added SW8_DP: SW_Push, PCM_Switch_Keyboard_Cherry_MX:SW_Cherry_MX_PCB, F.Cu at (60.0, 72.0)
- added TP1: TestPoint, TestPoint:TestPoint_THTPad_1.0x1.0mm_Drill0.5mm, F.Cu at (59.8, 35.6)
- added TP2: TestPoint, TestPoint:TestPoint_THTPad_1.0x1.0mm_Drill0.5mm, F.Cu at (73.9, 38.5)
- added TP3: TestPoint, TestPoint:TestPoint_Pad_D1.0mm, F.Cu at (86.4, 26.7)
- added TP4: TestPoint, TestPoint:TestPoint_Pad_D1.0mm, F.Cu at (84.1, 26.7)
- moved C16 79.0 mm to (81.7, 30.9)
- moved C11 77.4 mm to (71.9, 35.4)
- moved C12 77.4 mm to (81.6, 43.7)
- moved C13 77.4 mm to (86.4, 42.9)
- moved C14 77.4 mm to (91.3, 36.8)
- moved C4 77.4 mm to (95.9, 33.7)
- moved C6 77.4 mm to (78.9, 32.9)
- moved C7 77.4 mm to (78.9, 31.9)
- moved C8 77.4 mm to (91.3, 35.4)
- moved J1 77.4 mm to (76.4, 23.7)
- moved JP1 77.4 mm to (139.1, 47.2)
- moved JP10 77.4 mm to (139.1, 103.0)
- moved JP11 77.4 mm to (139.1, 106.0)
- moved JP12 77.4 mm to (139.1, 109.0)
- moved JP13 77.4 mm to (139.1, 112.0)
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- renumbered SW16_SPACE1 to SW16_SPACE
Connections:
- U1 pad 27: /Main/A2 -> /Main/P1
- U1 pad 28: /Main/A1 -> /Main/P2
- U1 pad 29: /Main/S1 -> /Main/P3
- U1 pad 30: /Main/S2 -> /Main/P4
- U1 pad 31: unconnected-(U1-GPIO20-Pad31) -> /Main/A2
- U1 pad 32: unconnected-(U1-GPIO21-Pad32) -> /Main/A1
- U1 pad 34: unconnected-(U1-GPIO22-Pad34) -> /Main/S1
- U1 pad 35: unconnected-(U1-GPIO23-Pad35) -> /Main/S2
- U1 pad 37: unconnected-(U1-GPIO25-Pad37) -> Net-(U1-GPIO25)
- U1 pad 39: unconnected-(U1-GPIO27_ADC1-Pad39) -> Net-(U1-GPIO27_ADC1)
Routing:
- net /Main/P4: track 0.00 -> 27.4 mm
- net /Main/P3: track 0.00 -> 23.8 mm
- net /Main/P2: track 0.00 -> 20.4 mm
- net /Main/P1: track 0.00 -> 17.6 mm
- net Net-(D1-K): track 0.00 -> 10.0 mm
- net Net-(U1-GPIO25): track 0.00 -> 7.94 mm
- net Net-(U1-GPIO27_ADC1): track 0.00 -> 7.08 mm
- net /Main/S1: track 53.9 -> 59.1 mm
- net +1V1: track 20.7 -> 25.8 mm
- net GND: track 230.5 -> 235.0 mm
- net /Main/S2: track 54.7 -> 58.9 mm
- net /Main/A1: track 54.0 -> 57.7 mm
- net /Main/A2: track 54.9 -> 58.0 mm
- net +3.3V: track 138.0 -> 141.1 mm
Other:
- outline, holes or cut-outs redrawn

Commit message: Add silkscreen images
Other:
- board text added: "GO AHEAD"
- board text added: "PEE"

Commit message: PCB Order Version
Parts:
- removed C16: 100n, Capacitor_SMD:C_0402_1005Metric
- removed C17, C18: 4.7u, Capacitor_SMD:C_0402_1005Metric
- removed the JP10 at (52.3, 110.4)
- removed the JP10 at (139.1, 103.0)
- removed the JP11 at (139.1, 106.0)
- removed the JP11 at (55.3, 110.4)
- removed the JP12 at (139.1, 109.0)
- removed the JP12 at (58.3, 110.4)
- removed the JP13 at (139.1, 112.0)
- removed the JP13 at (61.3, 110.4)
- removed the JP14 at (67.3, 110.4)
- removed the JP14 at (139.1, 118.0)
- removed the JP16 at (64.3, 110.4)
- removed the JP16 at (139.1, 115.0)
- removed the SW16_SPACE at (85.3, 99.1)
- removed the SW17_W at (117.1, 54.4)
- removed the SW18_DOWN at (109.8, 72.0)
- removed the SW19_LEFT at (92.2, 64.7)
- removed the SW20_RIGHT at (125.9, 83.0)
- removed the SW8_DP at (60.0, 72.0)
- added JP10: SolderJumper_2_Bridged, Fightstick_Library:EdgeSolderJumper-2_Right_Half, F.Cu at (52.3, 110.3)
- added JP10: SolderJumper_2_Bridged, Fightstick_Library:EdgeSolderJumper-2_Left_Half, F.Cu at (138.9, 103.0)
- added JP11: SolderJumper_2_Bridged, Fightstick_Library:EdgeSolderJumper-2_Right_Half, F.Cu at (55.3, 110.3)
- added JP11: SolderJumper_2_Bridged, Fightstick_Library:EdgeSolderJumper-2_Left_Half, F.Cu at (138.9, 106.0)
- added JP12: SolderJumper_2_Bridged, Fightstick_Library:EdgeSolderJumper-2_Right_Half, F.Cu at (58.3, 110.3)
- added JP12: SolderJumper_2_Bridged, Fightstick_Library:EdgeSolderJumper-2_Left_Half, F.Cu at (138.9, 109.0)
- added JP13: SolderJumper_2_Bridged, Fightstick_Library:EdgeSolderJumper-2_Left_Half, F.Cu at (138.9, 112.0)
- added JP13: SolderJumper_2_Bridged, Fightstick_Library:EdgeSolderJumper-2_Right_Half, F.Cu at (61.3, 110.3)
- added JP14: SolderJumper_2_Bridged, Fightstick_Library:EdgeSolderJumper-2_Right_Half, F.Cu at (67.3, 110.3)
- added JP14: SolderJumper_2_Bridged, Fightstick_Library:EdgeSolderJumper-2_Left_Half, F.Cu at (138.9, 118.0)
- added JP16: SolderJumper_2_Bridged, Fightstick_Library:EdgeSolderJumper-2_Left_Half, F.Cu at (138.9, 115.0)
- added JP16: SolderJumper_2_Bridged, Fightstick_Library:EdgeSolderJumper-2_Right_Half, F.Cu at (64.3, 110.3)
- added SW16_SPACE: SW_Push, PCM_Switch_Keyboard_Hotswap_Kailh:SW_Hotswap_Kailh_MX, F.Cu at (85.3, 99.1)
- added SW17_W: SW_Push, PCM_Switch_Keyboard_Hotswap_Kailh:SW_Hotswap_Kailh_MX_1.00u, F.Cu at (117.1, 54.4)
- added SW18_DOWN: SW_Push, PCM_Switch_Keyboard_Hotswap_Kailh:SW_Hotswap_Kailh_MX_1.00u, F.Cu at (109.8, 72.0)
- added SW19_LEFT: SW_Push, PCM_Switch_Keyboard_Hotswap_Kailh:SW_Hotswap_Kailh_MX_1.00u, F.Cu at (92.2, 64.7)
- added SW20_RIGHT: SW_Push, PCM_Switch_Keyboard_Hotswap_Kailh:SW_Hotswap_Kailh_MX_1.00u, F.Cu at (125.9, 83.0)
- added SW8_DP: SW_Push, PCM_Switch_Keyboard_Hotswap_Kailh:SW_Hotswap_Kailh_MX, F.Cu at (60.0, 72.0)
- added mouse-bite-2mm-slot: VAL**, Fightstick_Library:mouse-bite-2mm-slot, F.Cu at (97.4, 103.8)
- C1, C2: value 4.7u -> 10u
- D1, D2, D3, D4: footprint LED_SMD:LED_0603_1608Metric -> LED_SMD:LED_0805_2012Metric
- J1: footprint Fightstick_Library:USB_C_Receptacle_U262-161N-4BVC11 -> Fightstick_Library:USB_C_Receptacle_C6332272
- U2: footprint Package_TO_SOT_SMD:SOT-223-3_TabPin2 -> Fightstick_Library:LDO_AMS1117-3.3
- moved C11 10.8 mm to (81.7, 30.9)
- moved TP1 7.87 mm to (66.0, 30.8)
- moved mouse-bite-2mm-slot 6.95 mm to (97.4, 94.0)
- moved C2 5.70 mm to (72.0, 35.5), turned to 90 degrees
- moved R9 1.87 mm to (102.0, 38.0)
- moved C1 1.11 mm to (69.0, 31.0)
- moved JP17 0.15 mm to (52.3, 89.7)
- moved JP18 0.15 mm to (55.3, 89.7)
- moved JP19 0.15 mm to (58.3, 89.7)
- moved JP20 0.15 mm to (61.3, 89.7)
- moved JP1 0.14 mm to (138.9, 47.2)
- moved JP2 0.14 mm to (138.9, 28.0)
- moved JP3 0.14 mm to (138.9, 30.8)
- moved JP4 0.14 mm to (138.9, 33.5)
- moved JP5 0.14 mm to (138.9, 36.2)
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Connections:
- C2 pad 1: VBUS -> +3.3V
Routing:
- net +3.3V: track 141.1 -> 128.9 mm
- net L2: track 42.9 -> 48.2 mm, vias 0 -> 1
- net W: track 36.6 -> 33.1 mm, vias 0 -> 1
- net LEFT: track 23.1 -> 20.6 mm, vias 0 -> 1
- net DOWN: track 40.7 -> 38.2 mm, vias 0 -> 1
- net Net-(D1-K): track 10.0 -> 12.2 mm
- net /Buttons/SPACE: track 18.1 -> 17.0 mm, vias 0 -> 1
- net RIGHT: track 61.7 -> 60.7 mm, vias 0 -> 1
- net GND: track 235.0 -> 236.0 mm
Other:
- outline, holes or cut-outs redrawn
- board text removed: "JP17"
- board text removed: "JP18"
- board text removed: "JP19"
- board text removed: "JP20"
