File: KiCAD/4_board/panel_2.kicad_pcb (KiCad board)
At the start: 2 copper layers, 92.5 x 99.5 mm, 53 parts, among them SW10_SHARE1 SW_Push, SW11_START1 SW_Push, SW12_THROW1 SW_Push, SW14_PS1 SW_Push, SW15_TOUCHPAD1 SW_Push, SW2_LK1 SW_Push, SW3_MK1 SW_Push, SW4_LP1 SW_Push, SW5_MP1 SW_Push, SW6_DI1 SW_Push, SW7_HP1 SW_Push, SW9_HK1 SW_Push

Commit message: 4 board DFM pass
Parts:
- SW10_SHARE: renamed from SW10_SHARE1; footprint Button_Switch_THT:SW_SPST_Omron_B3F-40xx -> Fightstick_Library:SW_SPST_6x12
- SW11_START: renamed from SW11_START1; footprint Button_Switch_THT:SW_SPST_Omron_B3F-40xx -> Fightstick_Library:SW_SPST_6x12
- SW14_PS: renamed from SW14_PS1; footprint Button_Switch_THT:SW_SPST_Omron_B3F-40xx -> Fightstick_Library:SW_SPST_6x12
- SW15_TOUCHPAD: renamed from SW15_TOUCHPAD1; footprint Button_Switch_THT:SW_SPST_Omron_B3F-40xx -> Fightstick_Library:SW_SPST_6x12
- renumbered SW12_THROW1 to SW12_THROW, SW2_LK1 to SW2_LK, SW3_MK1 to SW3_MK, SW4_LP1 to SW4_LP, SW5_MP1 to SW5_MP, SW6_DI1 to SW6_DI, SW7_HP1 to SW7_HP, SW9_HK1 to SW9_HK
Changed lines of the file:
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@@
 		(descr "Cherry MX keyswitch PCB Mount")
 		(tags "Cherry MX Keyboard Keyswitch Switch PCB Cutout")
-		(property "Reference" "SW2_LK1"
+		(property "Reference" "SW2_LK"
 			(at 0 -8 0)
 			(unlocked yes)
@@
 		(descr "Cherry MX keyswitch PCB Mount")
 		(tags "Cherry MX Keyboard Keyswitch Switch PCB Cutout")
-		(property "Reference" "SW3_MK1"
+		(property "Reference" "SW3_MK"
 			(at 0 -8 0)
 			(unlocked yes)
@@
 		)
 	)
-	(footprint "Button_Switch_THT:SW_SPST_Omron_B3F-40xx"
+	(footprint "Fightstick_Library:SW_SPST_6x12"
 		(layer "F.Cu")
 		(at 170.08 55.05 90)
 		(descr "SW_THT_Tactile_Omron_B3F-40xx, 12x12 mm, Through hole switch from the B3F Family manufactured by Omron,  https://www.omron.com/ecb/products/pdf/en-b3f.pdf")
 		(tags "tactile switch THT button push B3F-4000 B3F-4050 B3F-4005 B3F-4055  ")
-		(property "Reference" "SW14_PS1"
-			(at 6.25 -4.5 90)
-			(unlocked yes)
+		(property "Reference" "SW14_PS"
+			(at 6.25 -4.5 270)
 			(layer "F.SilkS")
 			(effects
@@
 		(property "Value" "SW_Push"
 			(at 6.25 10.8 90)
-			(unlocked yes)
 			(layer "F.Fab")
 			(effects
@@
 			)
 		)
-		(property "Footprint" "Button_Switch_THT:SW_SPST_Omron_B3F-40xx"
+		(property "Footprint" "Fightstick_Library:SW_SPST_6x12"
 			(at 0 0 90)
 			(unlocked yes)
@@
 			)
 		)
-		(pad "" np_thru_hole circle
-			(at 6.25 -2 90)
-			(size 1.8 1.8)
-			(drill 1.8)
-			(layers "F&B.Cu" "*.Mask")
-		)
-		(pad "" np_thru_hole circle
-			(at 6.25 7 90)
-			(size 1.8 1.8)
-			(drill 1.8)
-			(layers "F&B.Cu" "*.Mask")
-		)
 		(pad "1" thru_hole oval
 			(at 0 0 90)
@@
 		(descr "Cherry MX keyswitch PCB Mount")
 		(tags "Cherry MX Keyboard Keyswitch Switch PCB Cutout")
-		(property "Reference" "SW4_LP1"
+		(property "Reference" "SW4_LP"
 			(at 0 -8 0)
 			(unlocked yes)
@@
 		)
 	)
-	(footprint "Button_Switch_THT:SW_SPST_Omron_B3F-40xx"
+	(footprint "Fightstick_Library:SW_SPST_6x12"
 		(layer "F.Cu")
 		(at 140.08 55.05 90)
 		(descr "SW_THT_Tactile_Omron_B3F-40xx, 12x12 mm, Through hole switch from the B3F Family manufactured by Omron,  https://www.omron.com/ecb/products/pdf/en-b3f.pdf")
 		(tags "tactile switch THT button push B3F-4000 B3F-4050 B3F-4005 B3F-4055  ")
-		(property "Reference" "SW11_START1"
-			(at 6.25 -4.5 90)
-			(unlocked yes)
+		(property "Reference" "SW11_START"
+			(at 6.25 -4.5 270)
 			(layer "F.SilkS")
 			(effects
@@
 		(property "Value" "SW_Push"
 			(at 6.25 10.8 90)
-			(unlocked yes)
 			(layer "F.Fab")
 			(effects
@@
 			)
 		)
-		(property "Footprint" "Button_Switch_THT:SW_SPST_Omron_B3F-40xx"
+		(property "Footprint" "Fightstick_Library:SW_SPST_6x12"
 			(at 0 0 90)
 			(unlocked yes)
@@
 			)
 		)
-		(pad "" np_thru_hole circle
-			(at 6.25 -2 90)
-			(size 1.8 1.8)
-			(drill 1.8)
-			(layers "F&B.Cu" "*.Mask")
-		)
-		(pad "" np_thru_hole circle
-			(at 6.25 7 90)
-			(size 1.8 1.8)
-			(drill 1.8)
-			(layers "F&B.Cu" "*.Mask")
-		)
 		(pad "1" thru_hole oval
 			(at 0 0 90)
@@
 		(descr "Cherry MX keyswitch PCB Mount")
 		(tags "Cherry MX Keyboard Keyswitch Switch PCB Cutout")
-		(property "Reference" "SW9_HK1"
+		(property "Reference" "SW9_HK"
 			(at 0 -8 0)
 			(unlocked yes)
@@
 		(descr "Cherry MX keyswitch PCB Mount")
 		(tags "Cherry MX Keyboard Keyswitch Switch PCB Cutout")
-		(property "Reference" "SW5_MP1"
+		(property "Reference" "SW5_MP"
 			(at 0 -8 0)
 			(unlocked yes)
@@
 		(descr "Cherry MX keyswitch PCB Mount")
 		(tags "Cherry MX Keyboard Keyswitch Switch PCB Cutout")
-		(property "Reference" "SW7_HP1"
+		(property "Reference" "SW7_HP"
 			(at 0 -8 0)
 			(unlocked yes)
@@
 		)
 	)
-	(footprint "Button_Switch_THT:SW_SPST_Omron_B3F-40xx"
+	(footprint "Fightstick_Library:SW_SPST_6x12"
 		(layer "F.Cu")
 		(at 185.08 55.05 90)
 		(descr "SW_THT_Tactile_Omron_B3F-40xx, 12x12 mm, Through hole switch from the B3F Family manufactured by Omron,  https://www.omron.com/ecb/products/pdf/en-b3f.pdf")
 		(tags "tactile switch THT button push B3F-4000 B3F-4050 B3F-4005 B3F-4055  ")
-		(property "Reference" "SW15_TOUCHPAD1"
-			(at 6.25 -4.5 90)
-			(unlocked yes)
+		(property "Reference" "SW15_TOUCHPAD"
+			(at 6.25 -4.5 270)
 			(layer "F.SilkS")
 			(effects
@@
 		(property "Value" "SW_Push"
 			(at 6.25 10.8 90)
-			(unlocked yes)
 			(layer "F.Fab")
 			(effects
@@
 			)
 		)
-		(property "Footprint" "Button_Switch_THT:SW_SPST_Omron_B3F-40xx"
+		(property "Footprint" "Fightstick_Library:SW_SPST_6x12"
 			(at 0 0 90)
 			(unlocked yes)
@@
 			)
 		)
-		(pad "" np_thru_hole circle
-			(at 6.25 -2 90)
-			(size 1.8 1.8)
-			(drill 1.8)
-			(layers "F&B.Cu" "*.Mask")
-		)
-		(pad "" np_thru_hole circle
-			(at 6.25 7 90)
-			(size 1.8 1.8)
-			(drill 1.8)
-			(layers "F&B.Cu" "*.Mask")
-		)
 		(pad "1" thru_hole oval
 			(at 0 0 90)
@@
 		(descr "Cherry MX keyswitch PCB Mount")
 		(tags "Cherry MX Keyboard Keyswitch Switch PCB Cutout")
-		(property "Reference" "SW12_THROW1"
+		(property "Reference" "SW12_THROW"
 			(at 0 -8 90)
 			(unlocked yes)
@@
 		(descr "Cherry MX keyswitch PCB Mount")
 		(tags "Cherry MX Keyboard Keyswitch Switch PCB Cutout")
-		(property "Reference" "SW6_DI1"
+		(property "Reference" "SW6_DI"
 			(at 0 -8 0)
 			(unlocked yes)
@@
 		)
 	)
-	(footprint "Button_Switch_THT:SW_SPST_Omron_B3F-40xx"
+	(footprint "Fightstick_Library:SW_SPST_6x12"
 		(layer "F.Cu")
 		(at 155.08 55.05 90)
 		(descr "SW_THT_Tactile_Omron_B3F-40xx, 12x12 mm, Through hole switch from the B3F Family manufactured by Omron,  https://www.omron.com/ecb/products/pdf/en-b3f.pdf")
 		(tags "tactile switch THT button push B3F-4000 B3F-4050 B3F-4005 B3F-4055  ")
-		(property "Reference" "SW10_SHARE1"
-			(at 6.25 -4.5 90)
-			(unlocked yes)
+		(property "Reference" "SW10_SHARE"
+			(at 6.25 -4.5 270)
 			(layer "F.SilkS")
 			(effects
@@
 		(property "Value" "SW_Push"
 			(at 6.25 10.8 90)
-			(unlocked yes)
 			(layer "F.Fab")
 			(effects
@@
 			)
 		)
-		(property "Footprint" "Button_Switch_THT:SW_SPST_Omron_B3F-40xx"
+		(property "Footprint" "Fightstick_Library:SW_SPST_6x12"
 			(at 0 0 90)
 			(unlocked yes)
@@
 			)
 		)
-		(pad "" np_thru_hole circle
-			(at 6.25 -2 90)
-			(size 1.8 1.8)
-			(drill 1.8)
-			(layers "F&B.Cu" "*.Mask")
-		)
-		(pad "" np_thru_hole circle
-			(at 6.25 7 90)
-			(size 1.8 1.8)
-			(drill 1.8)
-			(layers "F&B.Cu" "*.Mask")
-		)
 		(pad "1" thru_hole oval

Commit message: PCB Order Version
Parts:
- removed the JP15 at (102.5, 61.0)
- removed the JP15 at (165.8, 118.5)
- removed the JP21 at (102.5, 41.8)
- removed the JP21 at (146.6, 118.5)
- removed the JP22 at (102.5, 44.5)
- removed the JP22 at (149.3, 118.5)
- removed the JP23 at (102.5, 47.3)
- removed the JP23 at (152.1, 118.5)
- removed the JP24 at (154.8, 118.5)
- removed the JP24 at (102.5, 50.0)
- removed the JP25 at (102.5, 52.8)
- removed the JP25 at (157.6, 118.5)
- removed the JP26 at (102.5, 55.5)
- removed the JP26 at (160.3, 118.5)
- removed the JP27 at (102.5, 58.3)
- removed the JP27 at (163.1, 118.5)
- removed the SW10_SHARE at (155.1, 55.0)
- removed the SW11_START at (140.1, 55.0)
- removed the SW12_THROW at (178.9, 128.5)
- removed the SW14_PS at (170.1, 55.0)
- removed the SW15_TOUCHPAD at (185.1, 55.0)
- removed the SW2_LK at (117.5, 117.8)
- removed the SW3_MK at (142.5, 103.8)
- removed the SW4_LP at (117.5, 88.8)
- removed the SW5_MP at (142.5, 74.8)
- removed the SW6_DI at (117.7, 59.8)
- removed the SW7_HP at (171.5, 74.8)
- removed the SW9_HK at (171.5, 103.8)
- removed the mouse-bite-2mm-slot at (180.5, 117.8)
- removed the mouse-bite-2mm-slot at (170.0, 117.8)
- removed the mouse-bite-2mm-slot at (191.8, 117.8)
- added JP15: SolderJumper_2_Bridged, Fightstick_Library:EdgeSolderJumper-2_Left_Half, F.Cu at (158.8, 113.5)
- added JP15: SolderJumper_2_Bridged, Fightstick_Library:EdgeSolderJumper-2_Right_Half, F.Cu at (102.6, 61.0)
- added JP21: SolderJumper_2_Bridged, Fightstick_Library:EdgeSolderJumper-2_Right_Half, F.Cu at (102.6, 41.8)
- added JP21: SolderJumper_2_Bridged, Fightstick_Library:EdgeSolderJumper-2_Left_Half, F.Cu at (139.6, 113.5)
- added JP22: SolderJumper_2_Bridged, Fightstick_Library:EdgeSolderJumper-2_Left_Half, F.Cu at (142.3, 113.5)
- added JP22: SolderJumper_2_Bridged, Fightstick_Library:EdgeSolderJumper-2_Right_Half, F.Cu at (102.6, 44.5)
- added JP23: SolderJumper_2_Bridged, Fightstick_Library:EdgeSolderJumper-2_Left_Half, F.Cu at (145.1, 113.5)
- added JP23: SolderJumper_2_Bridged, Fightstick_Library:EdgeSolderJumper-2_Right_Half, F.Cu at (102.6, 47.3)
- added JP24: SolderJumper_2_Bridged, Fightstick_Library:EdgeSolderJumper-2_Left_Half, F.Cu at (147.8, 113.5)
- added JP24: SolderJumper_2_Bridged, Fightstick_Library:EdgeSolderJumper-2_Right_Half, F.Cu at (102.6, 50.0)
- added JP25: SolderJumper_2_Bridged, Fightstick_Library:EdgeSolderJumper-2_Right_Half, F.Cu at (102.6, 52.8)
- added JP25: SolderJumper_2_Bridged, Fightstick_Library:EdgeSolderJumper-2_Left_Half, F.Cu at (150.6, 113.5)
- added JP26: SolderJumper_2_Bridged, Fightstick_Library:EdgeSolderJumper-2_Right_Half, F.Cu at (102.6, 55.5)
- added JP26: SolderJumper_2_Bridged, Fightstick_Library:EdgeSolderJumper-2_Left_Half, F.Cu at (153.3, 113.5)
- added JP27: SolderJumper_2_Bridged, Fightstick_Library:EdgeSolderJumper-2_Right_Half, F.Cu at (102.6, 58.3)
- added JP27: SolderJumper_2_Bridged, Fightstick_Library:EdgeSolderJumper-2_Left_Half, F.Cu at (156.1, 113.5)
- added SW10_SHARE: SW_Push, PCM_Switch_Keyboard_Cherry_MX:SW_Cherry_MX_PCB, F.Cu at (155.1, 48.9)
- added SW11_START: SW_Push, PCM_Switch_Keyboard_Cherry_MX:SW_Cherry_MX_PCB, F.Cu at (139.6, 48.9)
- added SW12_THROW: SW_Push, PCM_Switch_Keyboard_Hotswap_Kailh:SW_Hotswap_Kailh_MX, F.Cu at (172.0, 123.4)
- added SW14_PS: SW_Push, PCM_Switch_Keyboard_Cherry_MX:SW_Cherry_MX_PCB, F.Cu at (170.6, 48.9)
- added SW15_TOUCHPAD: SW_Push, PCM_Switch_Keyboard_Cherry_MX:SW_Cherry_MX_PCB, F.Cu at (186.1, 48.9)
- added SW2_LK: SW_Push, PCM_Switch_Keyboard_Hotswap_Kailh:SW_Hotswap_Kailh_MX, F.Cu at (117.5, 117.8)
- added SW3_MK: SW_Push, PCM_Switch_Keyboard_Hotswap_Kailh:SW_Hotswap_Kailh_MX, F.Cu at (142.5, 103.8)
- added SW4_LP: SW_Push, PCM_Switch_Keyboard_Hotswap_Kailh:SW_Hotswap_Kailh_MX, F.Cu at (117.5, 88.8)
- added SW5_MP: SW_Push, PCM_Switch_Keyboard_Hotswap_Kailh:SW_Hotswap_Kailh_MX, F.Cu at (142.5, 74.8)
- added SW6_DI: SW_Push, PCM_Switch_Keyboard_Hotswap_Kailh:SW_Hotswap_Kailh_MX, F.Cu at (117.7, 59.8)
- added SW7_HP: SW_Push, PCM_Switch_Keyboard_Hotswap_Kailh:SW_Hotswap_Kailh_MX, F.Cu at (171.5, 74.8)
- added SW9_HK: SW_Push, PCM_Switch_Keyboard_Hotswap_Kailh:SW_Hotswap_Kailh_MX, F.Cu at (171.5, 103.8)
- added mouse-bite-2mm-slot: VAL**, Fightstick_Library:mouse-bite-2mm-slot, F.Cu at (184.8, 112.6)
- added mouse-bite-2mm-slot: VAL**, Fightstick_Library:mouse-bite-2mm-slot, F.Cu at (163.1, 112.6)
- added mouse-bite-2mm-slot: VAL**, Fightstick_Library:mouse-bite-2mm-slot, F.Cu at (167.3, 135.0)
- added mouse-bite-2mm-slot: VAL**, Fightstick_Library:mouse-bite-2mm-slot, F.Cu at (173.6, 112.6)
- added mouse-bite-2mm-slot: VAL**, Fightstick_Library:mouse-bite-2mm-slot, F.Cu at (184.6, 135.0)
- added mouse-bite-2mm-slot: VAL**, Fightstick_Library:mouse-bite-2mm-slot, F.Cu at (175.8, 135.0)
- added mouse-bite-2mm-slot: VAL**, Fightstick_Library:mouse-bite-2mm-slot, F.Cu at (189.0, 128.2)
- added mouse-bite-2mm-slot: VAL**, Fightstick_Library:mouse-bite-2mm-slot, F.Cu at (189.0, 119.2)
- moved JP1 8.73 mm to (158.8, 134.1)
- moved JP2 8.73 mm to (139.6, 134.1)
- moved JP3 8.73 mm to (142.3, 134.1)
- moved JP4 8.73 mm to (145.1, 134.1)
- moved JP5 8.73 mm to (147.8, 134.1)
- moved JP6 8.73 mm to (150.6, 134.1)
- moved JP7 8.73 mm to (153.3, 134.1)
- moved JP8 8.73 mm to (156.1, 134.1)
- moved JP9 8.73 mm to (161.7, 134.1)
- moved H6 8.66 mm to (183.6, 123.3)
- moved mouse-bite-2mm-slot 8.66 mm to (136.8, 117.8)
- moved mouse-bite-2mm-slot 8.66 mm to (136.8, 128.1)
- moved H7 8.42 mm to (143.4, 123.8)
- moved JP17 0.11 mm to (102.6, 116.8)
- moved JP18 0.11 mm to (102.6, 119.8)
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Routing:
- net GND: track 410.5 -> 333.9 mm, vias 1 -> 2
- net /Buttons/A1: track 84.5 -> 68.5 mm
- net /Buttons/A2: track 98.8 -> 83.3 mm
- net /Buttons/S2: track 49.7 -> 34.5 mm
- net /Buttons/S1: track 65.5 -> 54.1 mm
- net /Buttons/L1: track 13.0 -> 9.28 mm, vias 0 -> 1
- net /Buttons/B2: track 44.8 -> 41.5 mm, vias 0 -> 1
- net /Buttons/B4: track 41.3 -> 38.1 mm, vias 0 -> 1
- net /Buttons/R1: track 71.4 -> 68.5 mm, vias 0 -> 1
- net /Buttons/R2: track 76.3 -> 73.7 mm, vias 0 -> 1
- net /Buttons/B3: track 36.1 -> 33.5 mm, vias 0 -> 1
- net /Buttons/B1: track 15.8 -> 13.5 mm, vias 0 -> 1
- net /Buttons/L3: track 10.4 -> 9.05 mm, vias 0 -> 1
Other:
- outline, holes or cut-outs redrawn
- board text removed: "TODO Move these buttons further away from the rest"
