File: KiCAD/3_board/Main.kicad_sch (KiCad schematic)
At the start: 37 parts, among them J1 USB_C_Receptacle_USB2.0_14P, J2 Conn_01x03_Socket, SW1 Memory Reset, U1 RP2040, U2 AMS1117-3.3_SOT223, U3 W25Q128JVSIQ, Y1 12 mhz crystal

Commit message: Correct 27ohm resistor footprint to 0603 and add 10mm button
Parts:
- J1: JLCPCB_CORRECTION (none) -> 0; -0.8; 0
- R7, R8: footprint Resistor_SMD:R_0402_1005Metric -> Resistor_SMD:R_0603_1608Metric
- U2: JLCPCB_CORRECTION (none) -> 0; 0; 180
- U3: JLCPCB_CORRECTION (none) -> 0; 0; 270
Changed lines of the file:
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@@
 			)
 		)
-		(property "Footprint" "Resistor_SMD:R_0402_1005Metric"
+		(property "Footprint" "Resistor_SMD:R_0603_1608Metric"
 			(at 137.16 71.628 90)
 			(effects
@@
 			)
 		)
+		(property "JLCPCB_CORRECTION" "0; 0; 180"
+			(at 104.14 34.29 0)
+			(effects
+				(font
+					(size 1.27 1.27)
+				)
+				(hide yes)
+			)
+		)
 		(pin "2"
 		)
@@
 			)
 		)
-		(property "Footprint" "Resistor_SMD:R_0402_1005Metric"
+		(property "Footprint" "Resistor_SMD:R_0603_1608Metric"
 			(at 137.16 80.518 90)
 			(effects
@@
 			)
 		)
+		(property "JLCPCB_CORRECTION" "0; -0.8; 0"
+			(at 30.48 49.53 0)
+			(effects
+				(font
+					(size 1.27 1.27)
+				)
+				(hide yes)
+			)
+		)
 		(pin "B9"
 		)
@@
 			(at 78.74 167.64 0)
 			(effects
+				(font
+					(size 1.27 1.27)
+				)
+				(hide yes)
+			)
+		)
+		(property "JLCPCB_CORRECTION" "0; 0; 270"
+			(at 78.74 167.64 0)
+			(effects
