File: KiCAD/3_board - REV B/Main.kicad_sch (KiCad schematic)
At the start: 38 parts, among them J1 USB_C_Receptacle_USB2.0_14P, J2 Conn_01x03_Socket, J3 USB_A, SW1 Memory Reset, U1 RP2040, U2 AMS1117-3.3_SOT223, U3 W25Q128JVSIQ, Y1 12 mhz crystal

Commit message: Assembled Version
Connections:
- net +3.3V: now also R9.2
- net GND: no longer R9.2
- net P1: now also D1.1 (K); no longer D1.2 (A)
- net P2: now also D2.1 (K); no longer D2.2 (A)
- net P3: now also D3.1 (K); no longer D3.2 (A)
- net P4: now also D4.1 (K); no longer D4.2 (A)
- new net: D1.2 (A), D2.2 (A), D3.2 (A), D4.2 (A), R9.1
Other:
- moved on the sheet: D1, D2, D3, D4, R9
